File: pcb.kicad_pcb (KiCad board)
At the start: 2 copper layers, 80 x 35.4 mm, 40 parts, among them J1 USB_B_Micro, J2 BAT, J3 Conn_01x07, J4 PROG, SW1 MultiDirectionSwitch_5way, SW2 M1, SW3 M2, SW4 SW_Push_SPDT, SW5 M3, SW6 RST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

Commit message: cleanup schematic
Parts:
- JP1, JP2: value SolderJumper_3_Open -> (none)
